File: Keyboard/keyboard.kicad_pcb (KiCad board)
At the start: 2 copper layers, 100 x 100 mm, 60 parts, among them P1 CONN_01X05, SW1 SW_PUSH_SMALL, SW10 SW_PUSH_SMALL, SW11 SW_PUSH_SMALL, SW12 SW_PUSH_SMALL, SW13 SW_PUSH_SMALL, SW14 SW_PUSH_SMALL, SW15 SW_PUSH_SMALL, SW16 SW_PUSH_SMALL, SW17 SW_PUSH_SMALL, SW18 SW_PUSH_SMALL, SW19 SW_PUSH_SMALL, SW2 SW_PUSH_SMALL, SW20 SW_PUSH_SMALL, SW21 SW_PUSH_SMALL, SW22 SW_PUSH_SMALL, SW23 SW_PUSH_SMALL, SW24 SW_PUSH_SMALL, SW25 SW_PUSH_SMALL, SW3 SW_PUSH_SMALL, SW4 SW_PUSH_SMALL, SW5 SW_PUSH_SMALL, SW6 SW_PUSH_SMALL, SW7 SW_PUSH_SMALL, SW8 SW_PUSH_SMALL, SW9 SW_PUSH_SMALL, U1 ADP5589

Commit message: last of 1/3 size
Parts:
- removed LPC11U2x, REF**: QFN-32-1EP_7x7mm_Pitch0.65mm, DFN_QFN:QFN-32-1EP_7x7mm_Pitch0.65mm
- removed REF**: Pin_Header_Straight_1x05, Pin_Headers:Pin_Header_Straight_1x05
- removed REF**: USB_A, Connect:USB_A
- removed REF**: UQFN-48-1EP_6x6mm_Pitch0.4mm, DFN_QFN:UQFN-48-1EP_6x6mm_Pitch0.4mm
- removed SD1: MicroSD, local:MICRO_SD
- removed USB1: USB-MINI-B, local:USB_MICRO_B
- removed USB2640: QFN-48-1EP_7x7mm_Pitch0.5mm, DFN_QFN:QFN-48-1EP_7x7mm_Pitch0.5mm
- added C1: C, Capacitors_SMD:C_0603, F.Cu at (103.0, 59.5)
- added C2: C, Capacitors_SMD:C_0603, F.Cu at (101.5, 62.0)
- added C3: C, Capacitors_SMD:C_0603, F.Cu at (179.5, 70.5)
- added CON1: USB-MICRO-B, Connect:USB_Micro-B, F.Cu at (99.5, 57.0)
- added P2: GND, local:Pin_Header_Straight_1x01, F.Cu at (181.5, 126.5)
- added P3: +3v3, local:Pin_Header_Straight_1x01, F.Cu at (92.5, 108.5)
- added P4: +3v3, local:Pin_Header_Straight_1x01, F.Cu at (181.5, 107.5)
- added P5: SDA, local:Pin_Header_Straight_1x01, F.Cu at (187.5, 88.5)
- added P6: SDA, local:Pin_Header_Straight_1x01, F.Cu at (98.0, 88.5)
- added P7: SCL, local:Pin_Header_Straight_1x01, F.Cu at (98.5, 69.5)
- added P8: SCL, local:Pin_Header_Straight_1x01, F.Cu at (187.5, 70.0)
- added U2: APE8865N-33-HF-3, Housings_SOT-23_SOT-143_TSOT-6:SOT-23, F.Cu at (100.5, 59.5)
- P1: value CONN_01X05 -> GND; footprint Pin_Headers:Pin_Header_Angled_1x05 -> local:Pin_Header_Straight_1x01; moved to F.Cu
- moved P1 112.4 mm to (92.5, 126.5), turned to 0 degrees
- moved D25 5.00 mm to (175.0, 126.5)
- moved D4 4.00 mm to (99.0, 126.5)
- moved D1 3.50 mm to (105.5, 69.5)
- moved D24 3.50 mm to (167.0, 126.5)
- moved D20 3.00 mm to (158.0, 126.5)
- moved D5 3.00 mm to (107.0, 126.5)
- moved D19 2.00 mm to (150.0, 126.5)
- moved D23 2.00 mm to (173.0, 107.5)
- moved D9 2.00 mm to (116.0, 126.5)
- moved D10 1.00 mm to (124.0, 126.5)
- moved D15 1.00 mm to (141.0, 126.5)
Connections:
- U1 pad 17: +3.3V -> +3V3
- U1 pad 18: +3.3V -> +3V3
- U1 pad 22: Net-(P1-Pad4) -> Net-(CON1-Pad3)
- U1 pad 23: Net-(P1-Pad3) -> Net-(CON1-Pad2)
- U1 pad 24: Net-(P1-Pad2) -> (no net)
Routing:
- net +3V3: track 0.00 -> 244.9 mm, vias 0 -> 1
- net Net-(CON1-Pad3): track 0.00 -> 168.5 mm, vias 0 -> 1
- net Net-(CON1-Pad2): track 0.00 -> 120.9 mm, vias 0 -> 1
- net +3.3V: track 26.6 -> 0.00 mm
- net Net-(P1-Pad4): track 24.5 -> 0.00 mm
- net Net-(P1-Pad3): track 24.0 -> 0.00 mm
- net Net-(P1-Pad2): track 24.0 -> 0.00 mm
- net Net-(D10-Pad2): track 174.1 -> 186.3 mm
- net Net-(D14-Pad2): track 162.6 -> 153.0 mm
- net Net-(SW1-Pad1): track 178.8 -> 171.9 mm
- net Net-(D1-Pad2): track 80.6 -> 74.4 mm
- net (no net): track 5.03 -> 0.00 mm
- net Net-(C1-Pad1): track 0.00 -> 4.52 mm
- net GND: track 0.60 -> 5.02 mm, vias 1 -> 3
- net Net-(D1-Pad1): track 9.07 -> 12.6 mm
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Other:
- board size 100 x 100 mm -> 100 x 90 mm

Commit message: one piece
Parts:
- removed D7: DIODE, Diodes_SMD:Diode-SMA_Standard
- removed P1, P2: GND, local:Pin_Header_Straight_1x01
- removed P3, P4: +3v3, local:Pin_Header_Straight_1x01
- removed P5, P6: SDA, local:Pin_Header_Straight_1x01
- removed P7, P8: SCL, local:Pin_Header_Straight_1x01
- removed SW7: SW_PUSH_SMALL, Discret:SW_Matias_Quiet
- added D26: DIODE, Diodes_SMD:Diode-SMA_Standard, F.Cu at (162.0, 88.0)
- added D27: DIODE, Diodes_SMD:Diode-SMA_Standard, F.Cu at (165.0, 107.0)
- added D28: DIODE, Diodes_SMD:Diode-SMA_Standard, F.Cu at (140.0, 127.0)
- added D29: DIODE, Diodes_SMD:Diode-SMA_Standard, F.Cu at (311.0, 127.0)
- added D30: DIODE, Diodes_SMD:Diode-SMA_Standard, F.Cu at (317.0, 107.0)
- added D31: DIODE, Diodes_SMD:Diode-SMA_Standard, F.Cu at (295.0, 88.0)
- added D32: DIODE, Diodes_SMD:Diode-SMA_Standard, F.Cu at (285.0, 69.0)
- added D33: DIODE, Diodes_SMD:Diode-SMA_Standard, F.Cu at (171.0, 69.0)
- added D34: DIODE, Diodes_SMD:Diode-SMA_Standard, F.Cu at (181.0, 88.0)
- added D35: DIODE, Diodes_SMD:Diode-SMA_Standard, F.Cu at (172.0, 126.0)
- added D36: DIODE, Diodes_SMD:Diode-SMA_Standard, F.Cu at (131.0, 126.0)
- added D37: DIODE, Diodes_SMD:Diode-SMA_Standard, F.Cu at (302.0, 126.0)
- added D38: DIODE, Diodes_SMD:Diode-SMA_Standard, F.Cu at (298.0, 107.0)
- added D39: DIODE, Diodes_SMD:Diode-SMA_Standard, F.Cu at (276.0, 88.0)
- added D40: DIODE, Diodes_SMD:Diode-SMA_Standard, F.Cu at (266.0, 69.0)
- added D41: DIODE, Diodes_SMD:Diode-SMA_Standard, F.Cu at (190.0, 69.0)
- added D42: DIODE, Diodes_SMD:Diode-SMA_Standard, F.Cu at (184.0, 107.0)
- added D43: DIODE, Diodes_SMD:Diode-SMA_Standard, F.Cu at (188.0, 126.0)
- added D44: DIODE, Diodes_SMD:Diode-SMA_Standard, F.Cu at (150.0, 126.0)
- added D45: DIODE, Diodes_SMD:Diode-SMA_Standard, F.Cu at (292.0, 127.0)
- added D46: DIODE, Diodes_SMD:Diode-SMA_Standard, F.Cu at (279.0, 107.0)
- added D47: DIODE, Diodes_SMD:Diode-SMA_Standard, F.Cu at (257.0, 88.0)
- added D48: DIODE, Diodes_SMD:Diode-SMA_Standard, F.Cu at (247.0, 69.0)
- added D49: DIODE, Diodes_SMD:Diode-SMA_Standard, F.Cu at (209.0, 69.0)
- added D50: DIODE, Diodes_SMD:Diode-SMA_Standard, F.Cu at (203.0, 107.0)
- added D51: DIODE, Diodes_SMD:Diode-SMA_Standard, F.Cu at (210.0, 126.0)
- added D52: DIODE, Diodes_SMD:Diode-SMA_Standard, F.Cu at (159.0, 127.0)
- added D53: DIODE, Diodes_SMD:Diode-SMA_Standard, F.Cu at (283.0, 126.0)
- added D54: DIODE, Diodes_SMD:Diode-SMA_Standard, F.Cu at (260.0, 107.0)
- added D55: DIODE, Diodes_SMD:Diode-SMA_Standard, F.Cu at (238.0, 88.0)
- added D56: DIODE, Diodes_SMD:Diode-SMA_Standard, F.Cu at (228.0, 69.0)
- added D57: DIODE, Diodes_SMD:Diode-SMA_Standard, F.Cu at (200.0, 88.0)
- added D58: DIODE, Diodes_SMD:Diode-SMA_Standard, F.Cu at (222.0, 107.0)
- added D59: DIODE, Diodes_SMD:Diode-SMA_Standard, F.Cu at (226.0, 126.0)
- added D60: DIODE, Diodes_SMD:Diode-SMA_Standard, F.Cu at (197.0, 127.0)
- added D61: DIODE, Diodes_SMD:Diode-SMA_Standard, F.Cu at (267.0, 126.0)
- added D62: DIODE, Diodes_SMD:Diode-SMA_Standard, F.Cu at (248.0, 126.0)
- added D63: DIODE, Diodes_SMD:Diode-SMA_Standard, F.Cu at (241.0, 107.0)
- added D64: DIODE, Diodes_SMD:Diode-SMA_Standard, F.Cu at (219.0, 88.0)
- added SW26: SW_PUSH_SMALL, Discret:SW_Matias_Quiet, F.Cu at (165.0, 83.0)
- added SW27: SW_PUSH_SMALL, Discret:SW_Matias_Quiet, F.Cu at (168.0, 102.0)
- added SW28: SW_PUSH_SMALL, Discret:SW_Matias_Quiet, F.Cu at (134.0, 132.0)
- added SW29: SW_PUSH_SMALL, Discret:SW_Matias_Quiet, F.Cu at (305.0, 132.0)
- added SW30: SW_PUSH_SMALL, Discret:SW_Matias_Quiet, F.Cu at (320.0, 102.0)
- added SW31: SW_PUSH_SMALL, Discret:SW_Matias_Quiet, F.Cu at (298.0, 83.0)
- added SW32: SW_PUSH_SMALL, Discret:SW_Matias_Quiet, F.Cu at (288.0, 64.0)
- added SW33: SW_PUSH_SMALL, Discret:SW_Matias_Quiet, F.Cu at (174.0, 64.0)
- added SW34: SW_PUSH_SMALL, Discret:SW_Matias_Quiet, F.Cu at (184.0, 83.0)
- added SW35: SW_PUSH_SMALL, Discret:SW_Matias_Quiet, F.Cu at (175.0, 121.0)
- added SW36: SW_PUSH_SMALL, Discret:SW_Matias_Quiet, F.Cu at (137.0, 121.0)
- added SW37: SW_PUSH_SMALL, Discret:SW_Matias_Quiet, F.Cu at (308.0, 121.0)
- added SW38: SW_PUSH_SMALL, Discret:SW_Matias_Quiet, F.Cu at (301.0, 102.0)
- added SW39: SW_PUSH_SMALL, Discret:SW_Matias_Quiet, F.Cu at (279.0, 83.0)
- added SW40: SW_PUSH_SMALL, Discret:SW_Matias_Quiet, F.Cu at (269.0, 64.0)
- added SW41: SW_PUSH_SMALL, Discret:SW_Matias_Quiet, F.Cu at (193.0, 64.0)
- added SW42: SW_PUSH_SMALL, Discret:SW_Matias_Quiet, F.Cu at (187.0, 102.0)
- added SW43: SW_PUSH_SMALL, Discret:SW_Matias_Quiet, F.Cu at (194.0, 121.0)
- added SW44: SW_PUSH_SMALL, Discret:SW_Matias_Quiet, F.Cu at (156.0, 121.0)
- added SW45: SW_PUSH_SMALL, Discret:SW_Matias_Quiet, F.Cu at (286.0, 132.0)
- added SW46: SW_PUSH_SMALL, Discret:SW_Matias_Quiet, F.Cu at (282.0, 102.0)
- added SW47: SW_PUSH_SMALL, Discret:SW_Matias_Quiet, F.Cu at (260.0, 83.0)
- added SW48: SW_PUSH_SMALL, Discret:SW_Matias_Quiet, F.Cu at (250.0, 64.0)
- added SW49: SW_PUSH_SMALL, Discret:SW_Matias_Quiet, F.Cu at (212.0, 64.0)
- added SW50: SW_PUSH_SMALL, Discret:SW_Matias_Quiet, F.Cu at (206.0, 102.0)
- added SW51: SW_PUSH_SMALL, Discret:SW_Matias_Quiet, F.Cu at (213.0, 121.0)
- added SW52: SW_PUSH_SMALL, Discret:SW_Matias_Quiet, F.Cu at (153.0, 132.0)
- added SW53: SW_PUSH_SMALL, Discret:SW_Matias_Quiet, F.Cu at (289.0, 121.0)
- added SW54: SW_PUSH_SMALL, Discret:SW_Matias_Quiet, F.Cu at (263.0, 102.0)
- added SW55: SW_PUSH_SMALL, Discret:SW_Matias_Quiet, F.Cu at (241.0, 83.0)
- added SW56: SW_PUSH_SMALL, Discret:SW_Matias_Quiet, F.Cu at (231.0, 64.0)
- added SW57: SW_PUSH_SMALL, Discret:SW_Matias_Quiet, F.Cu at (203.0, 83.0)
- added SW58: SW_PUSH_SMALL, Discret:SW_Matias_Quiet, F.Cu at (225.0, 102.0)
- added SW59: SW_PUSH_SMALL, Discret:SW_Matias_Quiet, F.Cu at (232.0, 121.0)
- added SW60: SW_PUSH_SMALL, Discret:SW_Matias_Quiet, F.Cu at (191.0, 132.0)
- added SW61: SW_PUSH_SMALL, Discret:SW_Matias_Quiet, F.Cu at (270.0, 121.0)
- added SW62: SW_PUSH_SMALL, Discret:SW_Matias_Quiet, F.Cu at (251.0, 121.0)
- added SW63: SW_PUSH_SMALL, Discret:SW_Matias_Quiet, F.Cu at (244.0, 102.0)
- added SW64: SW_PUSH_SMALL, Discret:SW_Matias_Quiet, F.Cu at (222.0, 83.0)
- moved C1 263.1 mm to (366.0, 65.5)
- moved C2 263.1 mm to (364.5, 68.0)
- moved U2 263.1 mm to (363.5, 65.5)
- moved CON1 258.5 mm to (358.0, 57.0)
- moved SW5 246.0 mm to (343.0, 132.0)
- moved D5 242.0 mm to (349.0, 127.0)
- moved SW14 226.3 mm to (358.0, 102.0), turned to 180 degrees
- moved D14 222.9 mm to (355.0, 107.0)
- moved D8 222.9 mm to (342.0, 69.0)
- moved SW8 222.0 mm to (345.0, 64.0), turned to 180 degrees
- moved C3 211.5 mm to (391.0, 69.0)
- moved SW15 206.9 mm to (336.0, 83.0), turned to 180 degrees
- moved D15 195.8 mm to (333.0, 88.0)
- moved D13 189.5 mm to (330.0, 127.0)
- moved SW13 184.0 mm to (324.0, 132.0)
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Connections:
- C1 pad 1: Net-(C1-Pad1) -> +3V3
- C2 pad 1: +3V3 -> Net-(C2-Pad1)
- CON1 pad 1: Net-(C1-Pad1) -> Net-(C2-Pad1)
- D11 pad 2: Net-(D1-Pad2) -> Net-(D11-Pad2)
- D15 pad 2: Net-(D10-Pad2) -> Net-(D15-Pad2)
- D16 pad 2: Net-(D1-Pad2) -> Net-(D16-Pad2)
- D17 pad 2: Net-(D12-Pad2) -> Net-(D1-Pad2)
- D18 pad 2: Net-(D13-Pad2) -> Net-(D10-Pad2)
- D19 pad 2: Net-(D14-Pad2) -> Net-(D11-Pad2)
- D2 pad 2: Net-(D12-Pad2) -> Net-(D10-Pad2)
- D20 pad 2: Net-(D10-Pad2) -> Net-(D12-Pad2)
- D21 pad 2: Net-(D1-Pad2) -> Net-(D13-Pad2)
- D22 pad 2: Net-(D12-Pad2) -> Net-(D14-Pad2)
- D23 pad 2: Net-(D13-Pad2) -> Net-(D15-Pad2)
- D24 pad 2: Net-(D14-Pad2) -> Net-(D16-Pad2)
- D25 pad 2: Net-(D10-Pad2) -> Net-(D1-Pad2)
- D3 pad 2: Net-(D13-Pad2) -> Net-(D11-Pad2)
- D4 pad 2: Net-(D14-Pad2) -> Net-(D12-Pad2)
- D5 pad 2: Net-(D10-Pad2) -> Net-(D13-Pad2)
- D6 pad 2: Net-(D1-Pad2) -> Net-(D14-Pad2)
- D8 pad 2: Net-(D13-Pad2) -> Net-(D16-Pad2)
- D9 pad 2: Net-(D14-Pad2) -> Net-(D1-Pad2)
- SW11 pad 1: Net-(SW11-Pad1) -> Net-(SW10-Pad1)
- SW12 pad 1: Net-(SW11-Pad1) -> Net-(SW10-Pad1)
- SW13 pad 1: Net-(SW11-Pad1) -> Net-(SW10-Pad1)
- SW14 pad 1: Net-(SW11-Pad1) -> Net-(SW10-Pad1)
- SW15 pad 1: Net-(SW11-Pad1) -> Net-(SW10-Pad1)
- SW16 pad 1: Net-(SW16-Pad1) -> Net-(SW10-Pad1)
- SW17 pad 1: Net-(SW16-Pad1) -> Net-(SW17-Pad1)
- SW18 pad 1: Net-(SW16-Pad1) -> Net-(SW17-Pad1)
- SW19 pad 1: Net-(SW16-Pad1) -> Net-(SW17-Pad1)
- SW20 pad 1: Net-(SW16-Pad1) -> Net-(SW17-Pad1)
- SW21 pad 1: Net-(SW21-Pad1) -> Net-(SW17-Pad1)
- SW22 pad 1: Net-(SW21-Pad1) -> Net-(SW17-Pad1)
- SW23 pad 1: Net-(D23-Pad1) -> Net-(SW17-Pad1)
- SW23 pad 2: Net-(SW21-Pad1) -> Net-(D23-Pad1)
- SW24 pad 1: Net-(SW21-Pad1) -> Net-(SW17-Pad1)
- SW25 pad 1: Net-(SW21-Pad1) -> Net-(SW25-Pad1)
- SW6 pad 1: Net-(SW10-Pad1) -> Net-(SW1-Pad1)
- SW8 pad 1: Net-(SW10-Pad1) -> Net-(SW1-Pad1)
- U1 pad 10: (no net) -> Net-(D15-Pad2)
- U1 pad 12: Net-(D12-Pad2) -> Net-(D10-Pad2)
- U1 pad 13: Net-(D13-Pad2) -> Net-(D11-Pad2)
- U1 pad 14: Net-(D14-Pad2) -> Net-(D12-Pad2)
- U1 pad 15: Net-(D10-Pad2) -> Net-(D13-Pad2)
- U1 pad 16: (no net) -> Net-(D16-Pad2)
- U1 pad 3: Net-(SW11-Pad1) -> Net-(SW17-Pad1)
- U1 pad 4: Net-(SW21-Pad1) -> Net-(SW33-Pad1)
- U1 pad 5: Net-(SW16-Pad1) -> Net-(SW25-Pad1)
- U1 pad 6: (no net) -> Net-(SW41-Pad1)
- U1 pad 7: (no net) -> Net-(SW49-Pad1)
- U1 pad 8: (no net) -> Net-(SW57-Pad1)
- U1 pad 9: (no net) -> Net-(D14-Pad2)
- U2 pad 3: Net-(C1-Pad1) -> Net-(C2-Pad1)
Routing:
- net Net-(SW25-Pad1): track 0.00 -> 360.1 mm
- net Net-(SW1-Pad1): track 171.9 -> 521.2 mm
- net Net-(SW17-Pad1): track 0.00 -> 341.9 mm
- net Net-(SW33-Pad1): track 0.00 -> 337.9 mm
- net Net-(SW41-Pad1): track 0.00 -> 258.1 mm
- net Net-(SW49-Pad1): track 0.00 -> 245.0 mm
- net +3V3: track 244.9 -> 0.00 mm, vias 1 -> 0
- net Net-(SW10-Pad1): track 157.5 -> 385.5 mm
- net Net-(SW57-Pad1): track 0.00 -> 191.2 mm
- net Net-(CON1-Pad3): track 168.5 -> 0.00 mm, vias 1 -> 0
- net Net-(D11-Pad2): track 0.00 -> 161.4 mm
- net Net-(D16-Pad2): track 0.00 -> 150.8 mm
- net Net-(SW11-Pad1): track 136.1 -> 0.00 mm
- net Net-(D15-Pad2): track 0.00 -> 127.5 mm
- net Net-(CON1-Pad2): track 120.9 -> 0.00 mm, vias 1 -> 0
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- removed copper zone on B.Cu, net GND
- removed copper zone on F.Cu, net GND
Other:
- board size 100 x 90 mm -> 277 x 90 mm
